File: Electronics/Schematics/Switcher.sch (EAGLE design)
At the start: 26 parts, among them Q1 2N2222, Q2 BSS110, Q3 BSS296

Commit message: adjust mapping to micro
Connections:
- removed net ADC1: D1.C, R1.1, R2.2
- removed net ADC2: D4.C, R5.2, R6.1
- removed net ADC3: D5.C, R8.2, R9.1
- removed net P1.0: JP1.6
- removed net P1.1: JP1.5
- removed net P1.2: JP1.4
- new net P1.0_ADC1: D1.C, JP1.6, R1.1, R2.2
- new net P1.1_ADC2: D4.C, JP1.5, R5.2, R6.1
- new net P1.2_ADC3: D5.C, JP1.4, R8.2, R9.1
